Commit message: 241004

File: resources/robots/hi_cl_23_240925/urdf/hi_cl_23_240925_rl.urdf (robot description, URDF)
Before this commit: robot hi_cl_23_240925, 24 links, 23 joints
Links:
- link l_calf_link: geometry collision box size=0.012 0.06 0.1; visual mesh filename=../meshes/l_calf_link.STL
- link r_calf_link: geometry collision box size=0.012 0.06 0.1; visual mesh filename=../meshes/r_calf_link.STL
Joints:
- joint l_calf_joint: limit lower=-0.65 upper=1.65 effort=36 velocity=21 -> lower=-0.8 upper=1.5 effort=36 velocity=21; origin xyz=0 0 -0.10575 rpy=0 0.65 0 -> xyz=0 0 -0.10575 rpy=0 0.8 0
- joint l_hip_pitch_joint: limit lower=-1.25 upper=1.75 effort=36 velocity=21 -> lower=-1.1 upper=1.9 effort=36 velocity=21; origin xyz=0 0.02875 -0.06425 rpy=0 -0.25 0 -> xyz=0 0.02875 -0.06425 rpy=0 -0.4 0
- joint r_calf_joint: limit lower=-0.65 upper=1.65 effort=36 velocity=21 -> lower=-0.8 upper=1.5 effort=36 velocity=21; origin xyz=0 0 -0.10575 rpy=0 0.65 0 -> xyz=0 0 -0.10575 rpy=0 0.8 0
- joint r_hip_pitch_joint: limit lower=-1.25 upper=1.75 effort=36 velocity=21 -> lower=-1.1 upper=1.9 effort=36 velocity=21; origin xyz=0 -0.02875 -0.06425 rpy=0 -0.25 0 -> xyz=0 -0.02875 -0.06425 rpy=0 -0.4 0
